Commit message: Updated patrol_bot, removed robot.urdf.xacro

File: urdf/patrol_bot.urdf (robot description, URDF)
Before this commit: robot patrol_bot, 1 links, 0 joints
Links:
- added link addon_base; visual cylinder length=0.1 radius=0.05
- added link left_wheel; visual cylinder length=0.05 radius=0.05
- added link right_wheel; visual cylinder length=0.05 radius=0.05
- link base_link: geometry collision box size=0.5 0.2 0.1; visual box size=0.5 0.2 0.1
Joints:
- added joint addon_base_joint: type continuous, parent base_link, child addon_base, origin xyz=0 0 0.1 rpy=0 0 0
- added joint left_wheel_joint: type continuous, parent base_link, child left_wheel, origin xyz=0 -0.1 0 rpy=1.570 0 0
- added joint right_wheel_joint: type continuous, parent base_link, child right_wheel, origin xyz=0 0.1 0 rpy=1.570 0 0

Commit message: Updated robot model to 4-wheeled

File: urdf/patrol_bot.urdf (robot description, URDF)
Before this commit: robot patrol_bot, 4 links, 3 joints
Links:
- removed link left_wheel
- removed link right_wheel
- added link left_f_wheel; visual cylinder length=0.05 radius=0.05
- added link left_r_wheel; visual cylinder length=0.05 radius=0.05
- added link right_f_wheel; visual cylinder length=0.05 radius=0.05
- added link right_r_wheel; visual cylinder length=0.05 radius=0.05
Joints:
- removed joint left_wheel_joint
- removed joint right_wheel_joint
- added joint left_f_wheel_joint: type continuous, parent base_link, child left_f_wheel, origin xyz=0.15 -0.125 0 rpy=0 0 0, axis 0 1 0
- added joint left_r_wheel_joint: type continuous, parent base_link, child left_r_wheel, origin xyz=-0.15 -0.125 0 rpy=0 0 0, axis 0 1 0
- added joint right_f _wheel_joint: type continuous, parent base_link, child right_f_wheel, origin xyz=0.15 0.125 0 rpy=0 0 0, axis 0 1 0
- added joint right_r_wheel_joint: type continuous, parent base_link, child right_r_wheel, origin xyz=-0.15 0.125 0 rpy=0 0 0, axis 0 1 0
- joint addon_base_joint: axis (none) -> 0 0 1; limit (none) -> lower=-1.57 upper=1.57 effort=10 velocity=10; type continuous -> revolute
