Commit message: patrol_bot replaced by two new robot models (2wd and 4wd)

File: urdf/2wd_patrol_bot.urdf (robot description, URDF)
Before this commit: robot patrol_bot, 6 links, 5 joints
Links:
- removed link left_f_wheel
- removed link left_r_wheel
- removed link right_f_wheel
- removed link right_r_wheel
- added link base_footprint
- added link caster_wheel; visual sphere radius=0.05
- added link left_wheel; visual cylinder length=0.05 radius=0.1
- added link right_wheel; visual cylinder length=0.05 radius=0.1
- link base_link: geometry collision box size=0.6 0.4 0.2; visual box size=0.6 0.4 0.2
Joints:
- removed joint left_f_wheel_joint
- removed joint left_r_wheel_joint
- removed joint right_f _wheel_joint
- removed joint right_r_wheel_joint
- added joint base_joint: type fixed, parent base_footprint, child base_link, origin xyz=0 0 0.1 rpy=0 0 0
- added joint caster_wheel_joint: type fixed, parent base_link, child caster_wheel, origin xyz=0.15 0 -0.05 rpy=0 0 0
- added joint left_wheel_joint: type continuous, parent base_link, child left_wheel, origin xyz=-0.15 -0.225 0 rpy=0 0 0, axis 0 1 0
- added joint right_wheel_joint: type continuous, parent base_link, child right_wheel, origin xyz=-0.15 0.225 0 rpy=0 0 0, axis 0 1 0
- joint addon_base_joint: origin xyz=0 0 0.1 rpy=0 0 0 -> xyz=0 0 0.2 rpy=0 0 0
