Commit message: footprint link and joint added on 4wd_patrol_bot

File: urdf/4wd_patrol_bot.urdf (robot description, URDF)
Before this commit: robot 4wd_patrol_bot, 6 links, 5 joints
Links:
- added link base_footprint
Joints:
- added joint base_joint: type fixed, parent base_footprint, child base_link, origin xyz=0 0 0.05 rpy=0 0 0
